File: Temperature Monitor.kicad_pcb (KiCad board)
At the start: 2 copper layers, 60 x 60 mm, 25 parts, among them J1 Battery, J2 BME 280, J3 Display, SW1 Up, SW2 Down, SW3 Select, U2 XIAO-ESP32-C6-SMD

Commit message: Trying to get changes to be comitted
Parts:
- C1, C2: value 0.1U -> 0.1uF
- C3: value 0.1 -> 0.1uF
Changed lines of the file:
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@@
 			)
 		)
-		(property "Value" "0.1"
+		(property "Value" "0.1uF"
 			(at 1.25 3.75 90)
 			(layer "F.Fab")
@@
 			)
 		)
-		(property "Value" "0.1U"
+		(property "Value" "0.1uF"
 			(at 1.25 3.75 0)
 			(layer "F.Fab")
@@
 			)
 		)
-		(property "Value" "0.1U"
+		(property "Value" "0.1uF"
 			(at 1.25 3.75 0)
 			(layer "F.Fab")
@@
 	)
 	(segment
+		(start 148.2 100.289949)
+		(end 148.2 96.5)
+		(width 0.4)
+		(layer "F.Cu")
+		(net "/Down")
+	)
+	(segment
+		(start 151 91.31)
+		(end 151 93.7)
+		(width 0.4)
+		(layer "F.Cu")
+		(net "/Down")
+	)
+	(segment
+		(start 138.7166 107.9068)
+		(end 137 106.1902)
+		(width 0.4)
+		(layer "F.Cu")
+		(net "/Down")
+	)
+	(segment
+		(start 156.5 84)
+		(end 156.5 77.5)
+		(width 0.4)
+		(layer "F.Cu")
+		(net "/Down")
+	)
+	(segment
+		(start 138.0232 100.9768)
+		(end 138.5232 100.9768)
+		(width 0.4)
+		(layer "F.Cu")
+		(net "/Down")
+	)
+	(segment
+		(start 151 93.7)
+		(end 148.2 96.5)
+		(width 0.4)
+		(layer "F.Cu")
+		(net "/Down")
+	)
+	(segment
+		(start 138.8 100.7)
+		(end 147.789949 100.7)
+		(width 0.4)
+		(layer "F.Cu")
+		(net "/Down")
+	)
+	(segment
+		(start 137 106.1902)
+		(end 137 102)
+		(width 0.4)
+		(layer "F.Cu")
+		(net "/Down")
+	)
+	(segment
+		(start 151 91.31)
+		(end 151 89.5)
+		(width 0.4)
+		(layer "F.Cu")
+		(net "/Down")
+	)
+	(segment
+		(start 137 102)
+		(end 138.0232 100.9768)
+		(width 0.4)
+		(layer "F.Cu")
+		(net "/Down")
+	)
+	(segment
+		(start 138.5232 100.9768)
+		(end 138.8 100.7)
+		(width 0.4)
+		(layer "F.Cu")
+		(net "/Down")
+	)
+	(segment
+		(start 147.789949 100.7)
+		(end 148.2 100.289949)
+		(width 0.4)
+		(layer "F.Cu")
+		(net "/Down")
+	)
+	(segment
+		(start 151 89.5)
+		(end 156.5 84)
+		(width 0.4)
+		(layer "F.Cu")
+		(net "/Down")
+	)
+	(segment
 		(start 148.1 108.9283)
 		(end 151.5 108.9283)
@@
 	)
 	(segment
-		(start 160.81 97.5)
-		(end 164.5 97.5)
-		(width 0.4)
-		(layer "F.Cu")
-		(net "Net-(C2-Pad2)")
-	)
-	(segment
-		(start 151 83.69)
-		(end 151 79.294887)
-		(width 0.4)
-		(layer "F.Cu")
-		(net "Net-(C1-Pad2)")
-	)
-	(segment
-		(start 151 79.294887)
-		(end 150.205113 78.5)
-		(width 0.4)
-		(layer "F.Cu")
-		(net "Net-(C1-Pad2)")
-	)
-	(segment
-		(start 148.2 100.289949)
-		(end 148.2 96.5)
-		(width 0.4)
-		(layer "F.Cu")
-		(net "/Down")
-	)
-	(segment
-		(start 151 91.31)
-		(end 151 93.7)
-		(width 0.4)
-		(layer "F.Cu")
-		(net "/Down")
-	)
-	(segment
-		(start 138.7166 107.9068)
-		(end 137 106.1902)
-		(width 0.4)
-		(layer "F.Cu")
-		(net "/Down")
-	)
-	(segment
-		(start 156.5 84)
-		(end 156.5 77.5)
-		(width 0.4)
-		(layer "F.Cu")
-		(net "/Down")
-	)
-	(segment
-		(start 138.0232 100.9768)
-		(end 138.5232 100.9768)
-		(width 0.4)
-		(layer "F.Cu")
-		(net "/Down")
-	)
-	(segment
-		(start 151 93.7)
-		(end 148.2 96.5)
-		(width 0.4)
-		(layer "F.Cu")
-		(net "/Down")
-	)
-	(segment
-		(start 138.8 100.7)
-		(end 147.789949 100.7)
-		(width 0.4)
-		(layer "F.Cu")
-		(net "/Down")
-	)
-	(segment
-		(start 137 106.1902)
-		(end 137 102)
-		(width 0.4)
-		(layer "F.Cu")
-		(net "/Down")
-	)
-	(segment
-		(start 151 91.31)
-		(end 151 89.5)
-		(width 0.4)
-		(layer "F.Cu")
-		(net "/Down")
-	)
-	(segment
-		(start 137 102)
-		(end 138.0232 100.9768)
-		(width 0.4)
-		(layer "F.Cu")
-		(net "/Down")
-	)
-	(segment
-		(start 138.5232 100.9768)
-		(end 138.8 100.7)
-		(width 0.4)
-		(layer "F.Cu")
-		(net "/Down")
-	)
-	(segment
-		(start 147.789949 100.7)
-		(end 148.2 100.289949)
-		(width 0.4)
-		(layer "F.Cu")
-		(net "/Down")
-	)
-	(segment
-		(start 151 89.5)
-		(end 156.5 84)
-		(width 0.4)
-		(layer "F.Cu")
-		(net "/Down")
-	)
-	(segment
 		(start 153.19 96.31)
 		(end 156.5 93)
@@
 		(net "/Up")
 	)
+	(segment
+		(start 160.81 97.5)
+		(end 164.5 97.5)
+		(width 0.4)
+		(layer "F.Cu")
+		(net "Net-(C2-Pad2)")
+	)
+	(segment
+		(start 151 83.69)
+		(end 151 79.294887)
+		(width 0.4)
+		(layer "F.Cu")
+		(net "Net-(C1-Pad2)")
+	)
+	(segment
+		(start 151 79.294887)
+		(end 150.205113 78.5)
+		(width 0.4)
+		(layer "F.Cu")
+		(net "Net-(C1-Pad2)")
+	)
 	(zone
